Commit message: Deleted erratic description

File: x80sv_description/urdf/wheel.xacro (robot description, xacro)
@@ -5,5 +5,5 @@
     xmlns:controller="http://playerstage.sourceforge.net/gazebo/xmlschema/#controller"
     xmlns:interface="http://playerstage.sourceforge.net/gazebo/xmlschema/#interface">
-    <macro name="erratic_wheel" params="suffix parent *origin">
+    <macro name="wheel" params="suffix parent *origin">
         <joint name="${parent}_${suffix}_wheel_joint" type="continuous">
             <insert_block name="origin" />
@@ -26,5 +26,5 @@
                 <origin xyz="0 0 0" rpy="0 0 0" />
                 <geometry>
-                    <mesh filename="package://erratic_description/meshes/collada/erratic_front_wheel_link.dae"/>
+                    <mesh filename="package://x80sv_description/meshes/collada/erratic_front_wheel_link.dae"/>
                 </geometry>
                 <material name="Black" />
@@ -33,5 +33,5 @@
                 <origin xyz="0 0 0" rpy="0 0 0" />
                 <geometry>
-                    <mesh filename="package://erratic_description/meshes/collada/erratic_front_wheel_link.dae"/>
+                    <mesh filename="package://x80sv_description/meshes/collada/erratic_front_wheel_link.dae"/>
                 </geometry>
             </collision>

File: x80sv_description/urdf/x80sv.xacro (robot description, xacro)
@@ -1,5 +1,5 @@
 <?xml version='1.0' ?>
 <robot name="x80sv" xmlns:xacro="http://www.ros.org/wiki/xacro">
-	<xacro:include filename="$(find erratic_description)/urdf/erratic_wheel.xacro" />
+	<xacro:include filename="$(find x80sv_description)/urdf/wheel.xacro" />
  <!--
   Wheel inertia:
@@ -94,5 +94,5 @@
 			<origin xyz="0 0 -0.08" rpy="0 0 0" />
 			<geometry>
-				<mesh filename="package://erratic_description/meshes/collada/erratic_caster_support_link.dae"/>
+				<mesh filename="package://x80sv_description/meshes/collada/erratic_caster_support_link.dae"/>
 			</geometry>
 		</visual>
@@ -100,5 +100,5 @@
 			<origin xyz="0 0 0" rpy="0 0 0" />
 			<geometry>
-				<mesh filename="package://erratic_description/meshes/collada/erratic_caster_support_link.dae"/>
+				<mesh filename="package://x80sv_description/meshes/collada/erratic_caster_support_link.dae"/>
 			</geometry>
 		</collision>
@@ -129,5 +129,5 @@
 				<origin xyz="0 0 0" rpy="0 0 0" />
 				<geometry>
-					<mesh filename="package://erratic_description/meshes/collada/erratic_caster_wheel_link.dae"/>
+					<mesh filename="package://x80sv_description/meshes/collada/erratic_caster_wheel_link.dae"/>
 				</geometry>
 				<material name="Black"/>
@@ -136,5 +136,5 @@
 				<origin xyz="0 0 0" rpy="0 0 0" />
 				<geometry>
-					<mesh filename="package://erratic_description/meshes/collada/erratic_caster_wheel_link.dae"/>
+					<mesh filename="package://x80sv_description/meshes/collada/erratic_caster_wheel_link.dae"/>
 				</geometry>
 			</collision>
@@ -146,10 +146,10 @@
 		<kd  value="1.0" />
 	</gazebo>
-	<erratic_wheel suffix="left" parent="base_link">
+	<wheel suffix="left" parent="base_link">
 		<origin xyz="0.0 0.15525 -0.129" rpy="0 0 0" />
-	</erratic_wheel>
-	<erratic_wheel suffix="right" parent="base_link">
+	</wheel>
+	<wheel suffix="right" parent="base_link">
 		<origin xyz="0.0 -0.15525 -0.129" rpy="0 0 0" />
-	</erratic_wheel>
+	</wheel>
  <link name="laser_scanner">
   <collision>

Commit message: Added oscillation detection and filled in more gazebo parameters

File: x80sv_description/urdf/wheel.xacro (robot description, xacro)
@@ -42,8 +42,6 @@
             <kp  value="1000000.0" />
             <kd  value="1.0" />
-            <material>Erratic/Grey</material>
         </gazebo>
         <gazebo reference="${parent}_${suffix}_motor_link" >
-            <material>Erratic/White</material>
         </gazebo>
         <transmission type="pr2_mechanism_model/SimpleTransmission" name="${parent}_${suffix}_wheel_trans">

File: x80sv_description/urdf/x80sv.xacro (robot description, xacro)
@@ -226,9 +226,15 @@
 		<wheelSeparation>${wheel_distance}</wheelSeparation>
 		<wheelDiameter>${wheel_diameter}</wheelDiameter>
-		<torque>5</torque>
+		<wheelTorque>1</wheelTorque>
+		<wheelAcceleration>1</wheelAcceleration>
 		<commandTopic>cmd_vel</commandTopic>
 		<odometryTopic>odom</odometryTopic>
 		<odometryFrame>odom</odometryFrame>
 		<robotBaseFrame>base_footprint</robotBaseFrame>
+		<publishWheelTF>true</publishWheelTF>
+		<publishTf>1</publishTf>
+		<rosDebugLevel>na</rosDebugLevel>
+		<odometrySource>odom</odometrySource>
+		<publishWheelJointState>true</publishWheelJointState>
 	</plugin>
 </gazebo>
